File: pcb/minisumo_plusplus_2027/minisumo_plusplus_2027.kicad_pcb (KiCad board)
At the start: 2 copper layers, 240 x 148 mm, 10 parts, among them J3 Start Module - Conn_01x04_Pin, J5 Conn_01x10_Pin, J6 Start Module - Conn_01x04_Pin, SW1 SW_SPDT, U3 ESP32-C6-SuperMini

Commit message: ORDER - as ordered for prototyper! pcb schematic and layout touched up just before sending. 7.36eur 12-16d shipping estimate was to be produced by the 20th (sunday) so long as passes review.
Parts:
- removed A3: ~, minisumo_plusplus_2027:MT3608 DC-DC Boost Module – 28V 2A Step-Up Power Module
- removed the J6 at (42.9, 7.27)
- added A1: ~, minisumo_plusplus_2027:Mini_L298N_2_Channel_H_Bridge_DC_Motor_Driver_Board_with_MX1508-2.54_int1-4-special_silk, F.Cu at (151.7, 135.1)
- added A1: ~, minisumo_plusplus_2027:Mini_L298N_2_Channel_H_Bridge_DC_Motor_Driver_Board_with_MX1508-2.54_int1-4-special_silk, F.Cu at (228.2, 93.0)
- added A1: ~, minisumo_plusplus_2027:Mini_L298N_2_Channel_H_Bridge_DC_Motor_Driver_Board_with_MX1508-2.54_int1-4-special_silk, F.Cu at (151.7, 69.1)
- added A1: ~, minisumo_plusplus_2027:Mini_L298N_2_Channel_H_Bridge_DC_Motor_Driver_Board_with_MX1508-2.54_int1-4-special_silk, F.Cu at (151.7, 102.1)
- added A1: ~, minisumo_plusplus_2027:Mini_L298N_2_Channel_H_Bridge_DC_Motor_Driver_Board_with_MX1508-2.54_int1-4-special_silk, F.Cu at (228.2, 59.9)
- added A1: ~, minisumo_plusplus_2027:Mini_L298N_2_Channel_H_Bridge_DC_Motor_Driver_Board_with_MX1508-2.54_int1-4-special_silk, F.Cu at (228.2, 126.0)
- added A2: ~, minisumo_plusplus_2027:MT3608 DC-DC Boost Module – 28V 2A Step-Up Power Module, B.Cu at (207.1, 70.7)
- added A2: ~, minisumo_plusplus_2027:MT3608 DC-DC Boost Module – 28V 2A Step-Up Power Module, B.Cu at (207.1, 103.7)
- added A2: ~, minisumo_plusplus_2027:MT3608 DC-DC Boost Module – 28V 2A Step-Up Power Module, B.Cu at (207.1, 136.7)
- added A2: ~, minisumo_plusplus_2027:MT3608 DC-DC Boost Module – 28V 2A Step-Up Power Module, B.Cu at (12.2, 22.7)
- added A2: ~, minisumo_plusplus_2027:MT3608 DC-DC Boost Module – 28V 2A Step-Up Power Module, B.Cu at (172.8, 58.3)
- added A2: ~, minisumo_plusplus_2027:MT3608 DC-DC Boost Module – 28V 2A Step-Up Power Module, B.Cu at (172.8, 91.3)
- added A2: ~, minisumo_plusplus_2027:MT3608 DC-DC Boost Module – 28V 2A Step-Up Power Module, B.Cu at (172.8, 124.3)
- added J3: Start Module - Conn_01x04_Pin, Connector_PinHeader_2.54mm:PinHeader_1x04_P2.54mm_Vertical, F.Cu at (230.2, 90.8)
- added J3: Start Module - Conn_01x04_Pin, Connector_PinHeader_2.54mm:PinHeader_1x04_P2.54mm_Vertical, F.Cu at (149.7, 71.2)
- added J3: Start Module - Conn_01x04_Pin, Connector_PinHeader_2.54mm:PinHeader_1x04_P2.54mm_Vertical, F.Cu at (230.2, 57.8)
- added J3: Start Module - Conn_01x04_Pin, Connector_PinHeader_2.54mm:PinHeader_1x04_P2.54mm_Vertical, F.Cu at (149.7, 137.2)
- added J3: Start Module - Conn_01x04_Pin, Connector_PinHeader_2.54mm:PinHeader_1x04_P2.54mm_Vertical, F.Cu at (230.2, 123.8)
- added J3: Start Module - Conn_01x04_Pin, Connector_PinHeader_2.54mm:PinHeader_1x04_P2.54mm_Vertical, F.Cu at (149.7, 104.2)
- added J5: Conn_01x10_Pin, Connector_PinHeader_2.54mm:PinHeader_1x10_P2.54mm_Vertical, F.Cu at (153.5, 115.7)
- added J5: Conn_01x10_Pin, Connector_PinHeader_2.54mm:PinHeader_1x10_P2.54mm_Vertical, F.Cu at (153.5, 49.7)
- added J5: Conn_01x10_Pin, Connector_PinHeader_2.54mm:PinHeader_1x10_P2.54mm_Vertical, F.Cu at (226.4, 79.3)
- added J5: Conn_01x10_Pin, Connector_PinHeader_2.54mm:PinHeader_1x10_P2.54mm_Vertical, F.Cu at (153.5, 82.7)
- added J5: Conn_01x10_Pin, Connector_PinHeader_2.54mm:PinHeader_1x10_P2.54mm_Vertical, F.Cu at (226.4, 112.3)
- added J5: Conn_01x10_Pin, Connector_PinHeader_2.54mm:PinHeader_1x10_P2.54mm_Vertical, F.Cu at (226.4, 145.3)
- added J6: Start Module - Conn_01x04_Pin, minisumo_plusplus_2027:PinSocket_1x04_P2.54mm_Horizontal, F.Cu at (42.9, 7.26)
- added J6: Start Module - Conn_01x04_Pin, minisumo_plusplus_2027:PinSocket_1x04_P2.54mm_Horizontal, F.Cu at (237.9, 88.3)
- added J6: Start Module - Conn_01x04_Pin, minisumo_plusplus_2027:PinSocket_1x04_P2.54mm_Horizontal, F.Cu at (237.8, 121.3)
- added J6: Start Module - Conn_01x04_Pin, minisumo_plusplus_2027:PinSocket_1x04_P2.54mm_Horizontal, F.Cu at (237.9, 55.3)
- added J6: Start Module - Conn_01x04_Pin, minisumo_plusplus_2027:PinSocket_1x04_P2.54mm_Horizontal, F.Cu at (142.0, 106.7)
- added J6: Start Module - Conn_01x04_Pin, minisumo_plusplus_2027:PinSocket_1x04_P2.54mm_Horizontal, F.Cu at (142.1, 73.7)
- added J6: Start Module - Conn_01x04_Pin, minisumo_plusplus_2027:PinSocket_1x04_P2.54mm_Horizontal, F.Cu at (142.0, 139.8)
- added SW1: SW_SPDT, minisumo_plusplus_2027:SPST_switch_SS-12D00G4_1P2T_2.5mm_pitch_vert, F.Cu at (183.1, 140.8)
- added SW1: SW_SPDT, minisumo_plusplus_2027:SPST_switch_SS-12D00G4_1P2T_2.5mm_pitch_vert, F.Cu at (196.8, 87.2)
- added SW1: SW_SPDT, minisumo_plusplus_2027:SPST_switch_SS-12D00G4_1P2T_2.5mm_pitch_vert, F.Cu at (196.8, 54.2)
- added SW1: SW_SPDT, minisumo_plusplus_2027:SPST_switch_SS-12D00G4_1P2T_2.5mm_pitch_vert, F.Cu at (183.1, 74.8)
- added SW1: SW_SPDT, minisumo_plusplus_2027:SPST_switch_SS-12D00G4_1P2T_2.5mm_pitch_vert, F.Cu at (183.1, 107.8)
- added SW1: SW_SPDT, minisumo_plusplus_2027:SPST_switch_SS-12D00G4_1P2T_2.5mm_pitch_vert, F.Cu at (196.8, 120.2)
- added U2: ~, minisumo_plusplus_2027:battery cr123 3.7v with contacts for 18650_special_silk, B.Cu at (183.2, 78.2)
- added U2: ~, minisumo_plusplus_2027:battery cr123 3.7v with contacts for 18650_special_silk, B.Cu at (196.7, 116.8)
- added U2: ~, minisumo_plusplus_2027:battery cr123 3.7v with contacts for 18650_special_silk, B.Cu at (183.2, 144.2)
- added U2: ~, minisumo_plusplus_2027:battery cr123 3.7v with contacts for 18650_special_silk, B.Cu at (196.7, 83.8)
- added U2: ~, minisumo_plusplus_2027:battery cr123 3.7v with contacts for 18650_special_silk, B.Cu at (183.2, 111.2)
- added U2: ~, minisumo_plusplus_2027:battery cr123 3.7v with contacts for 18650_special_silk, B.Cu at (196.7, 50.8)
- added U3: ESP32-C6-SuperMini, minisumo_plusplus_2027:ESP32-C6-SuperMini_SMD_THT, F.Cu at (202.3, 90.7)
- added U3: ESP32-C6-SuperMini, minisumo_plusplus_2027:ESP32-C6-SuperMini_SMD_THT, F.Cu at (177.6, 137.3)
- added U3: ESP32-C6-SuperMini, minisumo_plusplus_2027:ESP32-C6-SuperMini_SMD_THT, F.Cu at (202.3, 123.7)
- added U3: ESP32-C6-SuperMini, minisumo_plusplus_2027:ESP32-C6-SuperMini_SMD_THT, F.Cu at (202.3, 57.7)
- added U3: ESP32-C6-SuperMini, minisumo_plusplus_2027:ESP32-C6-SuperMini_SMD_THT, F.Cu at (177.6, 104.3)
- added U3: ESP32-C6-SuperMini, minisumo_plusplus_2027:ESP32-C6-SuperMini_SMD_THT, F.Cu at (177.6, 71.3)
- U2: footprint BBQ_Library:battery cr123 3.7v with contacts for 18650 -> minisumo_plusplus_2027:battery cr123 3.7v with contacts for 18650_special_silk
Connections:
- A1 pad 2: Net-(A1-gnd) -> GND
- U3 pad 17: Net-(A1-INT3) -> Net-(A1-INT4)
- U3 pad 18: Net-(A1-INT4) -> Net-(A1-INT3)
Routing:
- net 3v3: track 77.8 -> 543.1 mm, vias 2 -> 14
- net GND: track 16.6 -> 390.8 mm, vias 7 -> 49
- net START Kill - not mandatory for sumo: track 30.9 -> 216.4 mm
- net IR Front: track 24.9 -> 182.6 mm, vias 1 -> 7
- net Net-(A1-INT1): track 26.4 -> 183.3 mm
- net IR Rear: track 28.3 -> 171.5 mm, vias 3 -> 21
- net Net-(A1-INT2): track 23.4 -> 162.1 mm
- net START Start: track 21.4 -> 150.1 mm
- net Net-(A1-INT4): track 18.9 -> 141.5 mm, vias 1 -> 7
- net /3v7 (>3v3 & <5v): track 18.8 -> 131.3 mm
- net Net-(A1-INT3): track 20.3 -> 115.9 mm, vias 1 -> 7
- net /9v: track 9.21 -> 64.4 mm
- net US Echo Tx: track 5.85 -> 40.9 mm
- net US Trigger Rx: track 5.85 -> 40.9 mm
- net Net-(SW1-A): track 3.27 -> 22.9 mm
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Other:
- board size 240 x 148 mm -> 241 x 147.1 mm
